File: PCB/strirling-measurement-PCB.kicad_pcb (KiCad board)
At the start: 2 copper layers, 25 parts, among them J1 NTC_Connector1, J2 NTC_Connector2, J3 NTC_Connector3, J4 NTC_Connector4, J5 NTC_Connector5, U1 NUCLEO-G431KB

Commit message: ready
Parts:
- removed C4, C5: 100nF, Capacitor_SMD:C_0805_2012Metric
- removed R10, R8: 1k, Resistor_SMD:R_0805_2012Metric
- removed R7, R9: 3.9k, Resistor_SMD:R_0603_1608Metric
- removed U1: NUCLEO-G431KB, stirling-measurement-PCB-footprintlibrary:MODULE_NUCLEO-G431KB
- added A1: RaspberryPi_Pico, Module:RaspberryPi_Pico_SMD_HandSolder, F.Cu at (100.0, 100.0)
- added TP1: NTC1, TestPoint:TestPoint_Pad_2.0x2.0mm, F.Cu at (119.0, 104.8)
- added TP2: NTC2, TestPoint:TestPoint_Pad_2.0x2.0mm, F.Cu at (119.0, 94.8)
- added TP3: NTC3, TestPoint:TestPoint_Pad_2.0x2.0mm, F.Cu at (119.0, 84.8)
- added TP4: 3v3_testpoint, TestPoint:TestPoint_Pad_2.0x2.0mm, F.Cu at (122.0, 115.0)
- added TP5: GND_testpoint, TestPoint:TestPoint_Pad_2.0x2.0mm, F.Cu at (122.0, 120.0)
- C1, C2, C3: footprint Capacitor_SMD:C_0805_2012Metric -> Capacitor_SMD:C_0402_1005Metric
- D1, D2: footprint LED_THT:LED_D5.0mm_FlatTop -> LED_THT:LED_D5.0mm
- J4: value NTC_Connector4 -> Gap-opto_module_socket; footprint stirling-measurement-PCB-footprintlibrary:JST_S2B-ZR_LF__SN_ -> stirling-measurement-PCB-footprintlibrary:gap-opto_module
- J5: value NTC_Connector5 -> SWD_socket; footprint stirling-measurement-PCB-footprintlibrary:JST_S2B-ZR_LF__SN_ -> stirling-measurement-PCB-footprintlibrary:swd_header
- R2, R4, R6: footprint Resistor_SMD:R_0805_2012Metric -> Resistor_SMD:R_0402_1005Metric
- moved R12 71.7 mm to (85.8, 98.7)
- moved J5 68.7 mm to (79.2, 109.2)
- moved R11 68.6 mm to (85.8, 88.6)
- moved D2 67.9 mm to (79.4, 98.7)
- moved D1 66.9 mm to (79.4, 88.6)
- moved C1 46.4 mm to (112.2, 99.2), turned to 90 degrees
- moved J4 43.1 mm to (104.3, 137.2), turned to -90 degrees
- moved C2 41.4 mm to (112.2, 96.7), turned to 90 degrees
- moved C3 34.6 mm to (112.2, 91.6), turned to 90 degrees
- moved R2 32.2 mm to (113.6, 98.7)
- moved J3 30.6 mm to (123.9, 85.6), turned to 90 degrees
- moved R4 28.0 mm to (113.6, 96.2)
- moved R1 23.0 mm to (116.6, 104.0), turned to 90 degrees
- moved R6 22.7 mm to (113.6, 91.1)
- moved J2 19.2 mm to (123.9, 95.6), turned to 90 degrees
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Connections:
- J4 pad 1: GND -> +3.3V
- J4 pad 2: Net-(J4-Pin_2) -> /GAP-OPTO_OUT
- J5 pad 1: GND -> /SWDIO
- J5 pad 2: Net-(J5-Pin_2) -> GND
- R12 pad 2: unconnected-(R12-Pad2) -> /USER2LED_GPIO
Routing:
- net /SWDIO: track 0.00 -> 30.9 mm, vias 0 -> 1
- net /SWCLK: track 0.00 -> 26.4 mm, vias 0 -> 1
- net GND: track 0.00 -> 26.0 mm, vias 0 -> 13
- net /GAP-OPTO_OUT: track 0.00 -> 17.9 mm
- net Net-(J1-Pin_2): track 0.00 -> 13.3 mm
- net Net-(J3-Pin_2): track 0.00 -> 13.0 mm
- net Net-(J2-Pin_2): track 0.00 -> 8.72 mm
- net +3.3V: track 0.00 -> 7.50 mm, vias 0 -> 5
- net /USER2LED_GPIO: track 0.00 -> 3.59 mm
- net /USER1LED_GPIO: track 0.00 -> 3.59 mm
- net /NTC3_ADC: track 0.00 -> 3.44 mm
- net /NTC2_ADC: track 0.00 -> 3.44 mm
- net /NTC1_ADC: track 0.00 -> 3.44 mm
- net Net-(D2-A): track 0.00 -> 2.91 mm
- net Net-(D1-A): track 0.00 -> 2.91 mm
- added copper zone on In2.Cu, net +3.3V
- added copper zone on In1.Cu, net GND
Other:
- board outline added: 50 x 65 mm
- copper layers 2 -> 4
- board text added: "3V3"
- board text added: "Dernovics Máté Dr. Csernovszky Zoltán Mihályffy Róbert"
- board text added: "Designed by:"
- board text added: "GND"
- board text added: "SIG"
- board text added: "SWCLK"
- board text added: "SWDIO"
- board text added: "Termistor 1"
- board text added: "Termistor 2"
- board text added: "Termistor 3"
- board text added: "User LED 1"
- board text added: "User LED 2"
